File: Hardware/main.kicad_sch (KiCad schematic)
At the start: 86 parts, among them J1 8x2 Character LCD, J2 Conn_01x16_Pin, J3 Conn_01x08_Pin, J4 Conn_02x05_Odd_Even, J5 Conn_01x02_Pin, J6 Conn_02x02_Odd_Even, J7 Conn_01x02_Pin, J8 Conn_01x02_Pin, J9 Conn_01x04_Pin, Q1 NPN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

Commit message: Changed LCD backlight resistance to 0
Parts:
- R5: value 510 -> 0
Changed lines of the file:
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@@
 			)
 		)
-		(property "Value" "510"
+		(property "Value" "0"
 			(at 329.692 134.112 90)
 			(effects
